File: Camera_Light/Led.sch (KiCad schematic (older format))
At the start: 18 parts, among them P1 CONN_01X03, P2 CONN_01X03

Commit message: defines.h wiederhergestellt
Changed lines of the file:
@@
 LIBS:valves
 LIBS:Led-cache
-EELAYER 25 0
+EELAYER 26 0
 EELAYER END
 $Descr A4 11693 8268
@@
 Text Label 1850 2650 3    60   ~ 0
 GREEN_VCC
+$Comp
+L PWR_FLAG #FLG05
+U 1 1 58B0233C
+P 7200 1650
+F 0 "#FLG05" H 7200 1745 50  0001 C CNN
+F 1 "PWR_FLAG" H 7200 1874 50  0000 C CNN
+F 2 "" H 7200 1650 50  0000 C CNN
+F 3 "" H 7200 1650 50  0000 C CNN
+	1    7200 1650
+	1    0    0    -1
+$EndComp
 $EndSCHEMATC
