File: Feeder_PCB/Feeder.kicad_pcb (KiCad board)
At the start: 2 copper layers, 49 parts, among them P1 CONN_01X04, P2 CONN_01X08, P3 CONN_01X01, P4 CONN_01X08, P5 CONN_02X03, P6 CONN_01X04, P7 CONN_01X03, U1 STM32_mmvisual_JTAG, U2 AP111733, U3 STM32F042K6Tx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

Commit message: code als submodul hinzugefügt
Parts:
- P1: value CONN_01X04 -> CONN_01X05; footprint Connectors_JST:JST_XH_B04B-XH-A_04x2.50mm_Straight -> Connectors_JST:JST_XH_B05B-XH-A_05x2.50mm_Straight
- P3: footprint Pin_Headers:Pin_Header_Angled_1x01_Pitch2.54mm -> Pin_Headers:Pin_Header_Straight_1x01_Pitch2.54mm
- P7: footprint Pin_Headers:Pin_Header_Angled_1x03_Pitch2.54mm -> Pin_Headers:Pin_Header_Straight_1x03_Pitch2.54mm
- moved D1 94.4 mm to (161.7, 53.6)
- moved C9 84.8 mm to (182.1, 84.8)
- moved C10 80.7 mm to (178.7, 95.3), turned to 270 degrees
- moved C11 78.5 mm to (180.6, 95.3), turned to 270 degrees
- moved U5 78.0 mm to (179.6, 90.6)
- moved C5 74.1 mm to (172.7, 96.2), turned to 270 degrees
- moved R15 73.1 mm to (182.1, 82.5)
- moved R16 72.1 mm to (175.6, 105.5), turned to 180 degrees
- moved R14 72.0 mm to (178.4, 82.5)
- moved P3 70.6 mm to (175.2, 82.5)
- moved C8 69.8 mm to (165.6, 105.3), turned to 90 degrees
- moved P6 69.4 mm to (179.9, 107.5), turned to 90 degrees
- moved C1 64.2 mm to (160.3, 57.1)
- moved C4 61.5 mm to (174.4, 96.2), turned to 270 degrees
- moved R12 57.7 mm to (159.3, 77.4), turned to 180 degrees
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Connections:
- P1 pad 1: /B -> /A
- P1 pad 2: /A -> /~A
- P1 pad 3: /~A -> /~B
- P1 pad 4: /~B -> /B
- U3 pad 12: /CAN_StandBy -> Net-(U3-Pad12)
- U3 pad 18: /~Enable -> /CAN_StandBy
- U3 pad 19: Net-(U3-Pad19) -> /~Enable
- U3 pad 20: Net-(U3-Pad20) -> /MS1
Routing:
- net +3V3: track 17.3 -> 139.9 mm, vias 2 -> 6
- net +5V: track 0.00 -> 106.3 mm, vias 0 -> 4
- net GND: track 41.5 -> 125.0 mm, vias 1 -> 12
- net /CAN_L: track 0.00 -> 50.8 mm, vias 0 -> 1
- net /CAN_H: track 0.00 -> 45.7 mm, vias 0 -> 1
- net /SwDIO: track 0.00 -> 31.2 mm, vias 0 -> 1
- net +24V: track 0.00 -> 29.0 mm, vias 0 -> 1
- net /ADC_MotorStrom: track 0.00 -> 28.8 mm, vias 0 -> 2
- net GNDPWR: track 0.00 -> 26.9 mm, vias 0 -> 1
- net /SwClk: track 0.00 -> 26.9 mm, vias 0 -> 1
- net /STM_DOut: track 0.00 -> 26.4 mm, vias 0 -> 1
- net /MS1: track 4.28 -> 28.2 mm, vias 0 -> 2
- net /~Enable: track 4.28 -> 26.8 mm, vias 0 -> 2
- net /ADC_LogicVcc: track 0.00 -> 22.2 mm
- net /ADC_PwrVcc: track 0.00 -> 21.4 mm, vias 0 -> 2
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- added copper zone on B.Cu, net GND
- added copper zone on F.Cu, net GND
Other:
- board outline added: 40 x 64 mm
- board text added: "DS18_20"
- board text added: "P.Hörauf 2017"
