File: Kopf_LED_Ring/Led.sch (KiCad schematic (older format))
At the start: 63 parts, among them IC1 AL8808, IC2 AL8808, IC3 AL8808, P1 CONN_01X04, P2 CONN_01X03, Q1 Q_NMOS_GSD

Commit message: neue Datenblätter, Wärmebilder vom weißen LichtRing und Software für den ComController
Parts:
- IC1, IC2, IC3: symbol DiodesInc:AL8808 -> Led-rescue:AL8808-DiodesInc
- P1: symbol conn:CONN_01X04 -> Led-rescue:CONN_01X04-conn
- P2: symbol conn:CONN_01X03 -> Led-rescue:CONN_01X03-conn
Other:
- note added: "vom Stecker aus runter:\n10% Power:\n1. 9,31mV\n2. 9,32mV\n3. 9,49mV\n\n30% Power:\n1. 27,85mV\n2. 27,87mV\n3. 28,65mV"
Changed lines of the file:
@@
 $EndComp
 $Comp
-L DiodesInc:AL8808 IC3
+L Led-rescue:AL8808-DiodesInc IC3
 U 1 1 5DDFDEEE
 P 1875 1875
@@
 $EndComp
 $Comp
-L DiodesInc:AL8808 IC1
+L Led-rescue:AL8808-DiodesInc IC1
 U 1 1 5DDFDF6F
 P 1850 2975
@@
 $EndComp
 $Comp
-L DiodesInc:AL8808 IC2
+L Led-rescue:AL8808-DiodesInc IC2
 U 1 1 5DDFEE92
 P 1850 4025
@@
 $EndComp
 $Comp
-L conn:CONN_01X04 P1
+L Led-rescue:CONN_01X04-conn P1
 U 1 1 5DE548B1
 P 2375 4950
@@
 $EndComp
 $Comp
-L conn:CONN_01X03 P2
+L Led-rescue:CONN_01X03-conn P2
 U 1 1 5DE96F1B
 P 4175 5900
@@
 	4950 6300 4950 6250
 Connection ~ 4950 6250
+Text Notes 8000 2300 0    50   ~ 0
+vom Stecker aus runter:\n10% Power:\n1. 9,31mV\n2. 9,32mV\n3. 9,49mV\n\n30% Power:\n1. 27,85mV\n2. 27,87mV\n3. 28,65mV
 $EndSCHEMATC
