File: LichtDom_SidePanels/LED_Panel_Hex.sch (KiCad schematic (older format))
At the start: 54 parts, among them P1 CONN_02X02, P2 CONN_02X02, Q1 Q_NPN_BEC, Q2 Q_NPN_BEC, Q3 Q_NPN_BEC, Q4 Q_NPN_BEC

Commit message: neue Datenblätter, Wärmebilder vom weißen LichtRing und Software für den ComController
Parts:
- H1, H2: symbol Mechanical:MountingHole -> LED_Panel_Hex-rescue:MountingHole-Mechanical
- P1, P2: symbol conn:CONN_02X02 -> LED_Panel_Hex-rescue:CONN_02X02-conn
Changed lines of the file:
@@
 CTRL_Red2
 $Comp
-L conn:CONN_02X02 P1
+L LED_Panel_Hex-rescue:CONN_02X02-conn P1
 U 1 1 5DE4CF3A
 P 8000 3075
@@
 CTRL_Red1
 $Comp
-L conn:CONN_02X02 P2
+L LED_Panel_Hex-rescue:CONN_02X02-conn P2
 U 1 1 5DE4E6B1
 P 7725 1400
@@
 Green_L2
 $Comp
-L Mechanical:MountingHole H1
+L LED_Panel_Hex-rescue:MountingHole-Mechanical H1
 U 1 1 5DE61D4E
 P 10375 1475
@@
 $EndComp
 $Comp
-L Mechanical:MountingHole H2
+L LED_Panel_Hex-rescue:MountingHole-Mechanical H2
 U 1 1 5DE61D9D
 P 10375 1675
